File: K40-LED_PCB/K40-LED_PCB.kicad_pcb (KiCad board)
At the start: 2 copper layers, 14 parts, among them p1 12V_Pad

Commit message: PCB_Update
Parts:
- moved D3 65.9 mm to (85.0, 68.0)
- moved D2 65.8 mm to (82.0, 65.0)
- moved D5 62.9 mm to (85.0, 78.0)
- moved D4 62.7 mm to (86.0, 73.0)
- moved D1 62.2 mm to (77.0, 64.0)
- moved D6 61.4 mm to (82.0, 80.7)
- moved D7 60.9 mm to (77.0, 82.0)
- moved D10 54.0 mm to (68.0, 73.0), turned to 180 degrees
- moved D12 2.25 mm to (127.8, 48.4)
- turned D11 to 150 degrees
- renumbered De to D11
Other:
- board outline added: 27.8 x 27.8 mm
Changed lines of the file:
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@@
   (general
     (thickness 1.6)
-    (drawings 0)
+    (drawings 2)
     (tracks 0)
     (zones 0)
@@
   )
   (module LRST-C190KGKT:LEDC1608X35N (layer F.Cu)
-    (at 129.38125 46.83125 120)
+    (at 127.79375 48.41875 120)
     (fp_text reference D12 (at 1.14732 -1.573661 120) (layer F.SilkS)
       (effects (font (size 1.002882 1.002882) (thickness 0.15)))
@@
   )
   (module LRST-C190KGKT:LEDC1608X35N (layer F.Cu)
-    (at 123.03125 50.8 180)
-    (fp_text reference De (at 1.14732 -1.573661) (layer F.SilkS)
+    (at 123.03125 50.8 150)
+    (fp_text reference D11 (at 1.14732 -1.573661 150) (layer F.SilkS)
+      (effects (font (size 1.002882 1.002882) (thickness 0.15)))
+    )
+    (fp_text value LTST-C190KGKT (at 5.60084 1.67287 150) (layer F.Fab)
+      (effects (font (size 1.002268 1.002268) (thickness 0.15)))
+    )
+    (fp_line (start 1.465 0.715) (end -1.465 0.715) (layer F.CrtYd) (width 0.05))
+    (fp_line (start 1.465 -0.715) (end 1.465 0.715) (layer F.CrtYd) (width 0.05))
+    (fp_line (start -1.465 -0.715) (end 1.465 -0.715) (layer F.CrtYd) (width 0.05))
+    (fp_line (start -1.465 0.715) (end -1.465 -0.715) (layer F.CrtYd) (width 0.05))
+    (fp_circle (center -2 0) (end -1.9 0) (layer F.Fab) (width 0.2))
+    (fp_circle (center -2 0) (end -1.9 0) (layer F.SilkS) (width 0.2))
+    (fp_line (start 0.85 0.45) (end -0.85 0.45) (layer F.Fab) (width 0.127))
+    (fp_line (start -0.85 -0.45) (end 0.85 -0.45) (layer F.Fab) (width 0.127))
+    (fp_line (start 0.085 0.45) (end -0.085 0.45) (layer F.SilkS) (width 0.127))
+    (fp_line (start 0.85 -0.45) (end 0.85 0.45) (layer F.Fab) (width 0.127))
+    (fp_line (start -0.085 -0.45) (end 0.085 -0.45) (layer F.SilkS) (width 0.127))
+    (fp_line (start -0.85 0.45) (end -0.85 -0.45) (layer F.Fab) (width 0.127))
+    (pad C smd rect (at -0.81 0 150) (size 0.81 0.93) (layers F.Cu F.Paste F.Mask)
+      (net 11 GND))
+    (pad A smd rect (at 0.81 0 150) (size 0.81 0.93) (layers F.Cu F.Paste F.Mask)
+      (net 9 "Net-(D11-PadA)"))
+  )
+  (module LRST-C190KGKT:LEDC1608X35N (layer F.Cu)
+    (at 68 73 180)
+    (fp_text reference D10 (at 1.14732 -1.573661) (layer F.SilkS)
       (effects (font (size 1.002882 1.002882) (thickness 0.15)))
     )
@@
     (fp_line (start 1.465 0.715) (end -1.465 0.715) (layer F.CrtYd) (width 0.05))
     (pad A smd rect (at 0.81 0 180) (size 0.81 0.93) (layers F.Cu F.Paste F.Mask)
-      (net 9 "Net-(D11-PadA)"))
+      (net 8 "Net-(D10-PadA)"))
     (pad C smd rect (at -0.81 0 180) (size 0.81 0.93) (layers F.Cu F.Paste F.Mask)
-      (net 11 GND))
-  )
-  (module LRST-C190KGKT:LEDC1608X35N (layer F.Cu)
-    (at 119.85625 57.94375)
-    (fp_text reference D10 (at 1.14732 -1.573661) (layer F.SilkS)
-      (effects (font (size 1.002882 1.002882) (thickness 0.15)))
-    )
-    (fp_text value LTST-C190KGKT (at 5.60084 1.67287) (layer F.Fab)
-      (effects (font (size 1.002268 1.002268) (thickness 0.15)))
-    )
-    (fp_line (start -0.85 0.45) (end -0.85 -0.45) (layer F.Fab) (width 0.127))
-    (fp_line (start -0.085 -0.45) (end 0.085 -0.45) (layer F.SilkS) (width 0.127))
-    (fp_line (start 0.85 -0.45) (end 0.85 0.45) (layer F.Fab) (width 0.127))
-    (fp_line (start 0.085 0.45) (end -0.085 0.45) (layer F.SilkS) (width 0.127))
-    (fp_line (start -0.85 -0.45) (end 0.85 -0.45) (layer F.Fab) (width 0.127))
-    (fp_line (start 0.85 0.45) (end -0.85 0.45) (layer F.Fab) (width 0.127))
-    (fp_circle (center -2 0) (end -1.9 0) (layer F.SilkS) (width 0.2))
-    (fp_circle (center -2 0) (end -1.9 0) (layer F.Fab) (width 0.2))
-    (fp_line (start -1.465 0.715) (end -1.465 -0.715) (layer F.CrtYd) (width 0.05))
-    (fp_line (start -1.465 -0.715) (end 1.465 -0.715) (layer F.CrtYd) (width 0.05))
-    (fp_line (start 1.465 -0.715) (end 1.465 0.715) (layer F.CrtYd) (width 0.05))
-    (fp_line (start 1.465 0.715) (end -1.465 0.715) (layer F.CrtYd) (width 0.05))
-    (pad A smd rect (at 0.81 0) (size 0.81 0.93) (layers F.Cu F.Paste F.Mask)
-      (net 8 "Net-(D10-PadA)"))
-    (pad C smd rect (at -0.81 0) (size 0.81 0.93) (layers F.Cu F.Paste F.Mask)
       (net 11 GND))
   )
@@
   )
   (module LRST-C190KGKT:LEDC1608X35N (layer F.Cu)
-    (at 136.525 69.05625 270)
+    (at 77 82 270)
     (fp_text reference D7 (at 1.14732 -1.573661 90) (layer F.SilkS)
       (effects (font (size 1.002882 1.002882) (thickness 0.15)))
@@
   )
   (module LRST-C190KGKT:LEDC1608X35N (layer F.Cu)
-    (at 142.08125 68.2625 300)
+    (at 82 80.701481 300)
     (fp_text reference D6 (at 1.14732 -1.573661 120) (layer F.SilkS)
       (effects (font (size 1.002882 1.002882) (thickness 0.15)))
@@
   )
   (module LRST-C190KGKT:LEDC1608X35N (layer F.Cu)
-    (at 146.05 62.70625 330)
+    (at 85 78 330)
     (fp_text reference D5 (at 1.14732 -1.573661 150) (layer F.SilkS)
       (effects (font (size 1.002882 1.002882) (thickness 0.15)))
@@
   )
   (module LRST-C190KGKT:LEDC1608X35N (layer F.Cu)
-    (at 146.84375 57.94375)
+    (at 86 73)
     (fp_text reference D4 (at 1.14732 -1.573661) (layer F.SilkS)
       (effects (font (size 1.002882 1.002882) (thickness 0.15)))
@@
   )
   (module LRST-C190KGKT:LEDC1608X35N (layer F.Cu)
-    (at 149.225 53.18125 30)
+    (at 85 68 30)
     (fp_text reference D3 (at 1.14732 -1.573661 30) (layer F.SilkS)
       (effects (font (size 1.002882 1.002882) (thickness 0.15)))
@@
   )
   (module LRST-C190KGKT:LEDC1608X35N (layer F.Cu)
-    (at 146.05 50.00625 60)
+    (at 82 65 60)
     (fp_text reference D2 (at 1.14732 -1.573661 60) (layer F.SilkS)
       (effects (font (size 1.002882 1.002882) (thickness 0.15)))
@@
   )
   (module LRST-C190KGKT:LEDC1608X35N (layer F.Cu)
-    (at 136.525 46.0375 90)
+    (at 77 64 90)
     (fp_text reference D1 (at 1.14732 -1.573661 90) (layer F.SilkS)
       (effects (font (size 1.002882 1.002882) (thickness 0.15)))
@@
       (net 2 "Net-(D1-PadC)"))
   )
+  (gr_circle (center 77 73) (end 89 80) (layer Edge.Cuts) (width 0.05))
+  (gr_circle (center 77 73) (end 82 73) (layer Edge.Cuts) (width 0.05))
 )

Commit message: PCB_Update
Parts:
- moved D8 60.2 mm to (72.0, 81.0)
- moved D12 58.2 mm to (72.0, 65.0)
- moved D11 56.7 mm to (69.0, 68.0)
- moved D9 55.0 mm to (69.0, 78.0)
- moved D6 0.30 mm to (82.0, 81.0)
Changed lines of the file:
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@@
   )
   (module LRST-C190KGKT:LEDC1608X35N (layer F.Cu)
-    (at 127.79375 48.41875 120)
+    (at 72 65 120)
     (fp_text reference D12 (at 1.14732 -1.573661 120) (layer F.SilkS)
       (effects (font (size 1.002882 1.002882) (thickness 0.15)))
@@
   )
   (module LRST-C190KGKT:LEDC1608X35N (layer F.Cu)
-    (at 123.03125 50.8 150)
+    (at 69 68 150)
     (fp_text reference D11 (at 1.14732 -1.573661 150) (layer F.SilkS)
       (effects (font (size 1.002882 1.002882) (thickness 0.15)))
@@
   )
   (module LRST-C190KGKT:LEDC1608X35N (layer F.Cu)
-    (at 122.2375 64.29375 210)
+    (at 69 78 210)
     (fp_text reference D9 (at 1.14732 -1.573661 30) (layer F.SilkS)
       (effects (font (size 1.002882 1.002882) (thickness 0.15)))
@@
   )
   (module LRST-C190KGKT:LEDC1608X35N (layer F.Cu)
-    (at 130.96875 69.05625 240)
+    (at 72 81 240)
     (fp_text reference D8 (at 1.14732 -1.573661 60) (layer F.SilkS)
       (effects (font (size 1.002882 1.002882) (thickness 0.15)))
@@
   )
   (module LRST-C190KGKT:LEDC1608X35N (layer F.Cu)
-    (at 82 80.701481 300)
+    (at 82 81 300)
     (fp_text reference D6 (at 1.14732 -1.573661 120) (layer F.SilkS)
       (effects (font (size 1.002882 1.002882) (thickness 0.15)))

Commit message: PCB_UPDATE
Parts:
- moved R1 68.2 mm to (97.0, 45.0)
Changed lines of the file:
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@@
   )
   (module Resistor_SMD:R_0805_2012Metric (layer F.Cu)
-    (at 164.315 55.995)
+    (at 97 45)
     (descr "Resistor SMD 0805 (2012 Metric), square (rectangular) end terminal, IPC_7351 nominal, (Body size source: IPC-SM-782 page 72, https://www.pcb-3d.com/wordpress/wp-content/uploads/ipc-sm-782a_amendment_1_and_2.pdf), generated with kicad-footprint-generator")
     (tags resistor)

Commit message: PCB_Update
Parts:
- moved D5 18.9 mm to (69.0, 68.0), turned to 150 degrees
- moved D12 18.4 mm to (85.0, 78.0), turned to 330 degrees
- moved D3 18.4 mm to (72.0, 81.0), turned to 240 degrees
- moved D10 18.0 mm to (86.0, 73.0), turned to 0 degrees
- moved D7 16.1 mm to (85.0, 68.0), turned to 30 degrees
- moved D9 13.3 mm to (82.0, 81.0), turned to 300 degrees
- moved D11 10.0 mm to (69.0, 78.0), turned to 210 degrees
- moved D2 9.00 mm to (73.0, 65.0), turned to 120 degrees
- moved D4 8.94 mm to (82.0, 65.0), turned to 60 degrees
- moved D8 8.94 mm to (68.0, 73.0), turned to 180 degrees
- moved D6 5.10 mm to (77.0, 82.0), turned to 270 degrees

Commit message: PCb_Complete
Parts:
- moved p1 47.8 mm to (102.7, 65.6), turned to 270 degrees
- moved R1 25.2 mm to (90.8, 69.4), turned to 90 degrees
- moved D2 1.00 mm to (72.0, 65.0)
Connections:
- D10 pad C: GND -> Net-(D10-PadC)
- D11 pad C: GND -> Net-(D10-PadC)
- D12 pad C: GND -> Net-(D10-PadC)
- p1 pad 2: Net-(p1-Pad2) -> Net-(D10-PadC)
Routing:
- net Net-(D1-PadA): track 0.00 -> 50.5 mm
- net Net-(D10-PadC): track 0.00 -> 33.1 mm
- net Net-(R1-Pad1): track 0.00 -> 7.19 mm
- net Net-(D5-PadC): track 0.00 -> 5.64 mm
- net Net-(D3-PadC): track 0.00 -> 5.64 mm
- net Net-(D10-PadA): track 0.00 -> 5.64 mm
- net Net-(D11-PadA): track 0.00 -> 5.62 mm
- net Net-(D6-PadC): track 0.00 -> 5.62 mm
- net Net-(D1-PadC): track 0.00 -> 5.62 mm
- net Net-(D2-PadC): track 0.00 -> 4.97 mm
- net Net-(D12-PadA): track 0.00 -> 4.89 mm
- net Net-(D4-PadC): track 0.00 -> 4.89 mm
Other:
- board size 27.8 x 27.8 mm -> 41 x 27.8 mm
- board text added: "NB's K40 LED"
